Commit message: right wheel added and it's joint

File: src/pibot_description/urdf/pibot.urdf.xacro (robot description, xacro)
@@ -15,3 +15,17 @@
         <origin xyz="0 0 0.033" rpy="0 0 0"/>
     </joint>
+    <link name="wheel_right_link">
+        <visual>
+            <origin xyz="0 0 0" rpy="0 0 0"/>
+            <geometry>
+                <mesh filename="package://pibot_description/meshes/wheel_right_link.STL"/>
+            </geometry>
+        </visual>
+    </link>
+    <joint name="wheel_right_joint" type="continuous">
+        <parent link="base_link"/>
+        <child link="wheel_right_link"/>
+        <axis xyz="0 1 0"/>
+        <origin xyz="0 -0.07 0" rpy="0 0 0"/>
+    </joint>
 </robot>
